File: cad/pcb/sensors.kicad_sch (KiCad schematic)
At the start: 9 parts

Commit message: generate bom; select C's & L's
Parts:
- C19: footprint (none) -> Capacitor_SMD:C_0603_1608Metric
- R22, R23, R24, R25: footprint (none) -> Resistor_SMD:R_0603_1608Metric
- TP12: footprint (none) -> TestPoint:TestPoint_Pad_D1.0mm
- V33: Mouser Part Number (none) -> PCA9957HNMP
- V34: footprint (none) -> Phototransistor:LEDC2012X95N; Mouser Part Number (none) -> SFH 3710-Z
Changed lines of the file:
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@@
   (symbol (lib_id "power:+3.3V") (at 82.55 45.72 0) (unit 1)
     (in_bom yes) (on_board yes)
-    (property "Reference" "#PWR072" (id 0) (at 82.55 49.53 0)
+    (property "Reference" "#PWR073" (id 0) (at 82.55 49.53 0)
       (effects (font (size 1.27 1.27)) hide)
     )
@@
   (symbol (lib_id "power:GND") (at 49.53 67.31 0) (unit 1)
     (in_bom yes) (on_board yes)
-    (property "Reference" "#PWR076" (id 0) (at 49.53 73.66 0)
+    (property "Reference" "#PWR077" (id 0) (at 49.53 73.66 0)
       (effects (font (size 1.27 1.27)) hide)
     )
@@
       (effects (font (size 1.27 1.27)) (justify left))
     )
-    (property "Footprint" "" (id 2) (at 90.17 120.65 0)
+    (property "Footprint" "Phototransistor:LEDC2012X95N" (id 2) (at 90.17 120.65 0)
       (effects (font (size 1.27 1.27)) hide)
     )
@@
       (effects (font (size 1.27 1.27)) hide)
     )
+    (property "Mouser Part Number" "SFH 3710-Z" (id 4) (at 85.09 123.19 0)
+      (effects (font (size 1.27 1.27)) hide)
+    )
     (pin "1")
     (pin "2")
@@
       (effects (font (size 1.27 1.27)) (justify left))
     )
-    (property "Footprint" "" (id 2) (at 170.18 69.85 0)
+    (property "Footprint" "Resistor_SMD:R_0603_1608Metric" (id 2) (at 170.18 69.85 0)
       (effects (font (size 1.27 1.27)) hide)
     )
@@
   (symbol (lib_id "power:+3.3V") (at 170.18 63.5 0) (unit 1)
     (in_bom yes) (on_board yes)
-    (property "Reference" "#PWR075" (id 0) (at 170.18 67.31 0)
+    (property "Reference" "#PWR076" (id 0) (at 170.18 67.31 0)
       (effects (font (size 1.27 1.27)) hide)
     )
@@
   (symbol (lib_id "power:GND") (at 87.63 143.51 0) (unit 1)
     (in_bom yes) (on_board yes)
-    (property "Reference" "#PWR081" (id 0) (at 87.63 149.86 0)
+    (property "Reference" "#PWR082" (id 0) (at 87.63 149.86 0)
       (effects (font (size 1.27 1.27)) hide)
     )
@@
       (effects (font (size 1.27 1.27)) (justify left))
     )
-    (property "Footprint" "" (id 2) (at 93.98 49.53 0)
+    (property "Footprint" "Resistor_SMD:R_0603_1608Metric" (id 2) (at 93.98 49.53 0)
       (effects (font (size 1.27 1.27)) hide)
     )
@@
       (effects (font (size 1.27 1.27)) (justify left))
     )
-    (property "Footprint" "" (id 2) (at 182.88 44.45 0)
+    (property "Footprint" "Resistor_SMD:R_0603_1608Metric" (id 2) (at 182.88 44.45 0)
       (effects (font (size 1.27 1.27)) hide)
     )
@@
   (symbol (lib_id "power:GND") (at 176.53 53.34 0) (unit 1)
     (in_bom yes) (on_board yes)
-    (property "Reference" "#PWR074" (id 0) (at 176.53 59.69 0)
+    (property "Reference" "#PWR075" (id 0) (at 176.53 59.69 0)
       (effects (font (size 1.27 1.27)) hide)
     )
@@
   (symbol (lib_id "power:GND") (at 82.55 67.31 0) (unit 1)
     (in_bom yes) (on_board yes)
-    (property "Reference" "#PWR077" (id 0) (at 82.55 73.66 0)
+    (property "Reference" "#PWR078" (id 0) (at 82.55 73.66 0)
       (effects (font (size 1.27 1.27)) hide)
     )
@@
   (symbol (lib_id "power:GND") (at 168.91 96.52 0) (unit 1)
     (in_bom yes) (on_board yes)
-    (property "Reference" "#PWR078" (id 0) (at 168.91 102.87 0)
+    (property "Reference" "#PWR079" (id 0) (at 168.91 102.87 0)
       (effects (font (size 1.27 1.27)) hide)
     )
@@
       (effects (font (size 1.27 1.27)) (justify left))
     )
-    (property "Footprint" "" (id 2) (at 82.55 62.23 0)
+    (property "Footprint" "Capacitor_SMD:C_0603_1608Metric" (id 2) (at 82.55 62.23 0)
       (effects (font (size 1.27 1.27)) hide)
     )
@@
     (property "Manufacturer_Part_Number" "PCA9957HNMP" (id 9) (at 212.09 76.2 0)
       (effects (font (size 1.27 1.27)) (justify left) hide)
+    )
+    (property "Mouser Part Number" "PCA9957HNMP" (id 10) (at 175.26 71.12 0)
+      (effects (font (size 1.27 1.27)) hide)
     )
     (pin "1")
@@
       (effects (font (size 1.27 1.27)) (justify left))
     )
-    (property "Footprint" "" (id 2) (at 87.63 135.89 0)
+    (property "Footprint" "Resistor_SMD:R_0603_1608Metric" (id 2) (at 87.63 135.89 0)
       (effects (font (size 1.27 1.27)) hide)
     )
@@
   (symbol (lib_id "power:GND") (at 222.25 96.52 0) (unit 1)
     (in_bom yes) (on_board yes)
-    (property "Reference" "#PWR079" (id 0) (at 222.25 102.87 0)
+    (property "Reference" "#PWR080" (id 0) (at 222.25 102.87 0)
       (effects (font (size 1.27 1.27)) hide)
     )
@@
       (effects (font (size 1.27 1.27)) (justify left))
     )
-    (property "Footprint" "" (id 2) (at 109.22 119.38 0)
+    (property "Footprint" "TestPoint:TestPoint_Pad_D1.0mm" (id 2) (at 109.22 119.38 0)
       (effects (font (size 1.27 1.27)) hide)
     )
@@
   (symbol (lib_id "power:+3.3V") (at 93.98 45.72 0) (unit 1)
     (in_bom yes) (on_board yes)
-    (property "Reference" "#PWR073" (id 0) (at 93.98 49.53 0)
+    (property "Reference" "#PWR074" (id 0) (at 93.98 49.53 0)
       (effects (font (size 1.27 1.27)) hide)
     )
@@
   (symbol (lib_id "power:+3.3V") (at 87.63 111.76 0) (unit 1)
     (in_bom yes) (on_board yes)
-    (property "Reference" "#PWR080" (id 0) (at 87.63 115.57 0)
-      (effects (font (size 1.27 1.27)) hide)
-    )
+    (property "Reference" "#PWR081" (id 0) (at 87.63 115.57 0)
+      (effects (font (size 1.27 1.27)) hide)
+    )
