File: pcb/mcu.kicad_sch (KiCad schematic)
At the start: 32 parts, among them X4 UART, X5 SWD, Y1 32MHz, Y2 32.768k

Commit message: add pcb fixes
Parts:
- X4: footprint myLib:PinHeader_P2mm_1x03_SMD -> myLib:PinHeader_2x03_P1.27mm_Vertical_SMD
Changed lines of the file:
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@@
       (effects (font (size 1.27 1.27)) (justify left))
     )
-    (property "Footprint" "myLib:PinHeader_P2mm_1x03_SMD" (id 2) (at 133.35 162.56 0)
+    (property "Footprint" "myLib:PinHeader_2x03_P1.27mm_Vertical_SMD" (id 2) (at 133.35 162.56 0)
       (effects (font (size 1.27 1.27)) hide)
     )
