File: pcb/power.kicad_sch (KiCad schematic)
At the start: 43 parts, among them X1 USB_C_Receptacle_USB2.0, X2 Bat-Conn, X3 NTC

Commit message: add pcb fixes
Connections:
- net GND: now also V3.1 (COMMON_A); no longer V2.7 (D2), V2.8 (D1), V3.2 (K_1)
- net VBUS_CONN: now also V3.2 (K_1); no longer V3.1 (COMMON_A)
- net at V2.3 (DRAIN2_1), V2.6 (DRAIN2_2): now also V2.7 (D2), V2.8 (D1)
Other:
- moved on the sheet: C4, C6, L2, R6, R7, TP7, TP8, V4
